File: rpi-adc-dac.kicad_pcb (KiCad board)
At the start: 2 copper layers, 5 parts, among them U1 rpi-pin-out

Commit message: update,
Parts:
- added C1: 105, Capacitor_SMD:C_0805_2012Metric_Pad1.15x1.40mm_HandSolder, B.Cu at (35.0, 40.9)
- added C2: 105, Capacitor_SMD:C_0805_2012Metric_Pad1.15x1.40mm_HandSolder, B.Cu at (42.5, 40.9)
- added C3: 105, Capacitor_SMD:C_0805_2012Metric_Pad1.15x1.40mm_HandSolder, B.Cu at (37.5, 40.9)
- added C4: 105, Capacitor_SMD:C_0805_2012Metric_Pad1.15x1.40mm_HandSolder, B.Cu at (40.0, 40.9)
- added C5: 105, Capacitor_SMD:C_0805_2012Metric_Pad1.15x1.40mm_HandSolder, B.Cu at (40.0, 36.0)
- added C6: 105, Capacitor_SMD:C_0805_2012Metric_Pad1.15x1.40mm_HandSolder, B.Cu at (42.5, 36.0)
- added C7: 105, Capacitor_SMD:C_0805_2012Metric_Pad1.15x1.40mm_HandSolder, B.Cu at (35.0, 36.0)
- added C8: 105, Capacitor_SMD:C_0805_2012Metric_Pad1.15x1.40mm_HandSolder, B.Cu at (37.5, 36.0)
- added D1: 3V3_STATUS, LED_SMD:LED_0805_2012Metric_Castellated, F.Cu at (29.0, 41.4)
- added D2: 5V_STATUS, LED_SMD:LED_0805_2012Metric_Castellated, F.Cu at (29.0, 36.9)
- added J1: Conn_01x02, Connector_PinSocket_2.54mm:PinSocket_1x06_P2.54mm_Vertical, F.Cu at (61.1, 70.9)
- added J2: Conn_01x02, Connector_PinSocket_2.54mm:PinSocket_1x02_P2.54mm_Vertical, F.Cu at (41.0, 45.2)
- added J3: Conn_01x02, Connector_PinSocket_2.54mm:PinSocket_1x10_P2.54mm_Vertical, F.Cu at (30.0, 72.5)
- added R1: 103, Resistor_SMD:R_0805_2012Metric_Pad1.15x1.40mm_HandSolder, F.Cu at (44.8, 44.0)
- added R10: R, Resistor_SMD:R_0805_2012Metric_Pad1.15x1.40mm_HandSolder, F.Cu at (36.0, 57.5)
- added R11: 103, Resistor_SMD:R_0805_2012Metric_Pad1.15x1.40mm_HandSolder, F.Cu at (36.0, 55.0)
- added R12: 103, Resistor_SMD:R_0805_2012Metric_Pad1.15x1.40mm_HandSolder, F.Cu at (47.2, 44.0)
- added R13: 682, Resistor_SMD:R_0805_2012Metric_Pad1.15x1.40mm_HandSolder, F.Cu at (43.5, 72.5)
- added R14: R, Resistor_SMD:R_0805_2012Metric_Pad1.15x1.40mm_HandSolder, F.Cu at (43.5, 69.9)
- added R15: 682, Resistor_SMD:R_0805_2012Metric_Pad1.15x1.40mm_HandSolder, F.Cu at (43.5, 67.5)
- added R16: 682, Resistor_SMD:R_0805_2012Metric_Pad1.15x1.40mm_HandSolder, F.Cu at (43.5, 65.0)
- added R17: 682, Resistor_SMD:R_0805_2012Metric_Pad1.15x1.40mm_HandSolder, F.Cu at (43.5, 62.5)
- added R18: 682, Resistor_SMD:R_0805_2012Metric_Pad1.15x1.40mm_HandSolder, F.Cu at (43.5, 60.0)
- added R19: 682, Resistor_SMD:R_0805_2012Metric_Pad1.15x1.40mm_HandSolder, F.Cu at (43.5, 57.5)
- added R2: 103, Resistor_SMD:R_0805_2012Metric_Pad1.15x1.40mm_HandSolder, F.Cu at (35.7, 36.5)
- added R20: 682, Resistor_SMD:R_0805_2012Metric_Pad1.15x1.40mm_HandSolder, F.Cu at (43.5, 55.0)
- added R21: 511, Resistor_SMD:R_0805_2012Metric_Pad1.15x1.40mm_HandSolder, F.Cu at (29.0, 39.2)
- added R22: 102, Resistor_SMD:R_0805_2012Metric_Pad1.15x1.40mm_HandSolder, F.Cu at (29.1, 34.6)
- added R3: 103, Resistor_SMD:R_0805_2012Metric_Pad1.15x1.40mm_HandSolder, F.Cu at (35.8, 34.0)
- added R4: 103, Resistor_SMD:R_0805_2012Metric_Pad1.15x1.40mm_HandSolder, F.Cu at (36.0, 72.5)
- added R5: 103, Resistor_SMD:R_0805_2012Metric_Pad1.15x1.40mm_HandSolder, F.Cu at (36.0, 69.9)
- added R6: 103, Resistor_SMD:R_0805_2012Metric_Pad1.15x1.40mm_HandSolder, F.Cu at (36.0, 67.5)
- added R7: 103, Resistor_SMD:R_0805_2012Metric_Pad1.15x1.40mm_HandSolder, F.Cu at (36.0, 65.0)
- added R8: 103, Resistor_SMD:R_0805_2012Metric_Pad1.15x1.40mm_HandSolder, F.Cu at (36.0, 62.5)
- added R9: 103, Resistor_SMD:R_0805_2012Metric_Pad1.15x1.40mm_HandSolder, F.Cu at (36.0, 60.0)
- added U2: MCP3424, Package_SO:SOIC-14_3.9x8.7mm_P1.27mm, F.Cu at (52.5, 70.0)
- added U3: FDC6301N, Package_TO_SOT_SMD:SuperSOT-6, F.Cu at (35.0, 46.3)
- added U4: MCP3424, Package_SO:SOIC-14_3.9x8.7mm_P1.27mm, F.Cu at (52.2, 58.2)
Connections:
- U1 pad 1: Net-(U1-Pad1) -> +3V3
- U1 pad 14: Net-(U1-Pad14) -> GND
- U1 pad 2: Net-(U1-Pad2) -> +5V
- U1 pad 20: Net-(U1-Pad20) -> GND
- U1 pad 25: Net-(U1-Pad25) -> GND
- U1 pad 3: Net-(U1-Pad3) -> /GPIO0
- U1 pad 30: Net-(U1-Pad30) -> GND
- U1 pad 34: Net-(U1-Pad34) -> GND
- U1 pad 39: Net-(U1-Pad39) -> GND
- U1 pad 5: Net-(U1-Pad5) -> /GPIO1
- U1 pad 6: Net-(U1-Pad6) -> GND
- U1 pad 9: Net-(U1-Pad9) -> GND
Routing:
- net +5V: track 0.00 -> 101.7 mm, vias 0 -> 6
- net Net-(R13-Pad2): track 0.00 -> 71.6 mm, vias 0 -> 2
- net GND: track 0.00 -> 47.5 mm, vias 0 -> 2
- net /SDA: track 0.00 -> 44.7 mm, vias 0 -> 1
- net /SCL: track 0.00 -> 38.4 mm, vias 0 -> 3
- net +3V3: track 0.00 -> 36.2 mm, vias 0 -> 1
- net Net-(R17-Pad1): track 0.00 -> 31.1 mm, vias 0 -> 2
- net Net-(R14-Pad1): track 0.00 -> 29.4 mm, vias 0 -> 2
- net Net-(J1-Pad4): track 0.00 -> 27.1 mm, vias 0 -> 2
- net Net-(R18-Pad1): track 0.00 -> 22.6 mm, vias 0 -> 2
- net /GPIO0: track 0.00 -> 22.4 mm, vias 0 -> 1
- net Net-(R16-Pad1): track 0.00 -> 22.2 mm, vias 0 -> 2
- net Net-(R13-Pad1): track 0.00 -> 21.3 mm
- net Net-(R11-Pad2): track 0.00 -> 20.3 mm
- net Net-(J1-Pad3): track 0.00 -> 18.4 mm, vias 0 -> 2
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- added copper zone on B.Cu, net GND
- added copper zone on F.Cu, net GND
