File: rpi-adc-dac.sch (KiCad schematic (older format))
At the start: 1 part, among them U1 rpi-pin-out

Commit message: update,
Parts:
- added C1, C2, C3, C4, C5, C6, C7, C8: 105, Capacitor_SMD:C_0805_2012Metric_Pad1.15x1.40mm_HandSolder, symbol Device:C
- added D1: 3V3_STATUS, LED_SMD:LED_0805_2012Metric_Castellated, symbol Device:LED
- added D2: 5V_STATUS, LED_SMD:LED_0805_2012Metric_Castellated, symbol Device:LED
- added J1: Conn_01x02, Connector_PinSocket_2.54mm:PinSocket_1x06_P2.54mm_Vertical, symbol Connector_Generic:Conn_01x06
- added J2: Conn_01x02, Connector_PinSocket_2.54mm:PinSocket_1x02_P2.54mm_Vertical, symbol Connector_Generic:Conn_01x02
- added J3: Conn_01x02, Connector_PinSocket_2.54mm:PinSocket_1x10_P2.54mm_Vertical, symbol Connector_Generic:Conn_01x10
- added R1, R11, R12, R2, R3, R4, R5, R6, R7, R8, R9: 103, Resistor_SMD:R_0805_2012Metric_Pad1.15x1.40mm_HandSolder, symbol Device:R
- added R10, R14: R, Resistor_SMD:R_0805_2012Metric_Pad1.15x1.40mm_HandSolder, symbol Device:R
- added R13, R15, R16, R17, R18, R19, R20: 682, Resistor_SMD:R_0805_2012Metric_Pad1.15x1.40mm_HandSolder, symbol Device:R
- added R21: 511, Resistor_SMD:R_0805_2012Metric_Pad1.15x1.40mm_HandSolder, symbol Device:R
- added R22: 102, Resistor_SMD:R_0805_2012Metric_Pad1.15x1.40mm_HandSolder, symbol Device:R
- added U2, U4: MCP3424, Package_SO:SOIC-14_3.9x8.7mm_P1.27mm, symbol Analog_ADC:MCP3424
- added U3: FDC6301N, Package_TO_SOT_SMD:SuperSOT-6, symbol taobao-components:FDC6301N
Connections:
- net labels added: +3V3, +5V, GND, GPIO0, GPIO1, SCL, SDA
- wire segments 0 -> 193

Commit message: update,
Parts:
- removed C1, C2, C3, C4, C5, C6, C7, C8: 105, Capacitor_SMD:C_0805_2012Metric_Pad1.15x1.40mm_HandSolder, symbol Device:C
- removed J1: Conn_01x02, Connector_PinSocket_2.54mm:PinSocket_1x06_P2.54mm_Vertical, symbol Connector_Generic:Conn_01x06
- removed J2: Conn_01x02, Connector_PinSocket_2.54mm:PinSocket_1x02_P2.54mm_Vertical, symbol Connector_Generic:Conn_01x02
- removed J3: Conn_01x02, Connector_PinSocket_2.54mm:PinSocket_1x10_P2.54mm_Vertical, symbol Connector_Generic:Conn_01x10
- removed R1, R11, R12, R2, R3, R4, R5, R6, R7, R8, R9: 103, Resistor_SMD:R_0805_2012Metric_Pad1.15x1.40mm_HandSolder, symbol Device:R
- removed R10, R14: R, Resistor_SMD:R_0805_2012Metric_Pad1.15x1.40mm_HandSolder, symbol Device:R
- removed R13, R15, R16, R17, R18, R19, R20: 682, Resistor_SMD:R_0805_2012Metric_Pad1.15x1.40mm_HandSolder, symbol Device:R
- removed U2, U4: MCP3424, Package_SO:SOIC-14_3.9x8.7mm_P1.27mm, symbol Analog_ADC:MCP3424
- removed U3: FDC6301N, Package_TO_SOT_SMD:SuperSOT-6, symbol taobao-components:FDC6301N
Connections:
- net labels removed: SCL, SDA
- wire segments 193 -> 28
Other:
- note added: "missing SCL and SDA"
